Commit message: fixing camera issues

File: catkin_ws/src/my_robot/urdf/my_robot.xacro (robot description, xacro)
@@ -201,5 +201,5 @@
   </link>
   <joint name="camera_joint" type="fixed">
-    <origin xyz="0.225 0 0.03" rpy="0 0 0"/>
+    <origin xyz="0.225 0 0.03" rpy="-1.5707 0 -1.5707"/>
     <parent link="chassis"/>
     <child link="camera"/>

Commit message: minors

File: catkin_ws/src/my_robot/urdf/my_robot.xacro (robot description, xacro)
@@ -201,5 +201,5 @@
   </link>
   <joint name="camera_joint" type="fixed">
-    <origin xyz="0.225 0 0.03" rpy="-1.5707 0 -1.5707"/>
+    <origin xyz="0.225 0 0.03" rpy="0 0 0"/>
     <parent link="chassis"/>
     <child link="camera"/>

Commit message: review finding fixing

File: catkin_ws/src/my_robot/urdf/my_robot.xacro (robot description, xacro)
@@ -206,4 +206,11 @@
     <axis xyz="0 1 0"/>
   </joint>
+  <joint name="camera_optical_joint" type="fixed">
+    <origin xyz="0 0 0" rpy="-1.5707 0 -1.5707"/>
+    <parent link="camera"/>
+    <child link="camera_link_optical"/>
+  </joint>
+  <link name="camera_link_optical">
+  </link>
   <link name='hokuyo'>
     <inertial>
